Commit message: robot car with fake_velocity

File: src/robot_description/urdf/robot.xacro (robot description, xacro)
@@ -8,5 +8,5 @@
     <inertial>
       <mass value="10.0"/>
-      <origin xyz="0.0 0 0.1" rpy=" 0 0 0"/>
+      <origin xyz="0.0 0 0.1" rpy="0 0 0"/>
       <inertia
           ixx="0.5" ixy="0" ixz="0"

Commit message: fixed all urdf and physical issues, tested with simple_control.py

File: src/robot_description/urdf/robot.xacro (robot description, xacro)
@@ -1,4 +1,6 @@
 <?xml version='1.0'?>
 <robot name="robot" xmlns:xacro="http://www.ros.org/wiki/xacro">
+  <xacro:property name="cameraSize" value="0.05"/>
+  <xacro:property name="cameraMass" value="0.1"/>
   <xacro:include filename="$(find robot_description)/urdf/robot.gazebo" />
   <xacro:include filename="$(find robot_description)/urdf/materials.xacro" />
@@ -7,6 +9,6 @@
     <pose>0 0 0.1 0 0 0</pose>
     <inertial>
-      <mass value="10.0"/>
-      <origin xyz="0.0 0 0.1" rpy="0 0 0"/>
+      <mass value="5.0"/>
+      <origin xyz="0.0 0 0.05" rpy="0 0 0"/>
       <inertia
           ixx="0.5" ixy="0" ixz="0"
@@ -17,54 +19,149 @@
     <collision name='collision'>
       <geometry>
-        <box size=".4 .2 .1"/>
+        <box size=".21 .2 .06"/>
       </geometry>
     </collision>
     <visual name='chassis_visual'>
-      <origin xyz="0 0 0" rpy=" 0 0 0"/>
-      <geometry>
-        <box size=".4 .2 .1"/>
-      </geometry>
-    </visual>
-    <collision name='caster_collision'>
-      <origin xyz="-0.15 0 -0.05" rpy=" 0 0 0"/>
-      <geometry>
-        <sphere radius="0.05"/>
-      </geometry>
-      <surface>
-        <friction>
-          <ode>
-            <mu>0</mu>
-            <mu2>0</mu2>
-            <slip1>1.0</slip1>
-            <slip2>1.0</slip2>
+      <origin xyz="0 0 0.05" rpy=" 0 0 0"/>
+      <geometry>
+        <box size=".21 .2 .06"/>
+      </geometry>
+    </visual>
+  </link>
+  <link name="left_wheel_front">
+    <!--origin xyz="0.1 0.13 0.1" rpy="0 1.5707 1.5707"/-->
+    <collision name="collision">
+      <origin xyz="0 0 0" rpy="0 1.5707 1.5707"/>
+      <geometry>
+        <cylinder radius="0.04" length="0.05"/>
+      </geometry>
+      <surface>
+        <friction>
+          <ode>
+            <mu>10</mu>
+            <mu2>10</mu2>
+          </ode>
+      </friction>
+      </surface>
+    </collision>
+    <visual name="left_wheel_front_visual">
+      <origin xyz="0 0 0" rpy="0 1.5707 1.5707"/>
+      <geometry>
+        <cylinder radius="0.04" length="0.04"/>
+      </geometry>
+    </visual>
+    <inertial>
+      <mass value="4"/>
+      <origin xyz="0 0 0" rpy="0 0 0"/>
+      <inertia
+          ixx="1.0" ixy="0" ixz="0"
+          iyy="1.0" iyz="0"
+          izz="1.0"
+      />
+    </inertial>
+  </link>
+  <link name="left_wheel_middle">
+    <!--origin xyz="0.1 0.13 0.1" rpy="0 1.5707 1.5707"/-->
+    <collision name="collision">
+      <origin xyz="0 0 0.008" rpy="0 1.5707 1.5707"/>
+      <geometry>
+        <box size=".075 .18 .04"/>
+      </geometry>
+    </collision>
+    <visual name="left_wheel_middle_visual">
+      <origin xyz="0 0 0.008" rpy="0 1.5707 1.5707"/>
+      <geometry>
+        <box size=".075 .18 .04"/>
+      </geometry>
+    </visual>
+    <inertial>
+      <origin xyz="0 0 0" rpy="0 1.5707 1.5707"/>
+      <mass value="2"/>
+      <inertia
+        ixx="1.0" ixy="0.0" ixz="0.0"
+        iyy="1.0" iyz="0.0"
+        izz="1.0"/>
+    </inertial>
+  </link>
+  <link name="left_wheel">
+    <!--origin xyz="0.1 0.13 0.1" rpy="0 1.5707 1.5707"/-->
+    <collision name="collision">
+      <origin xyz="0 0 0" rpy="0 1.5707 1.5707"/>
+      <geometry>
+        <cylinder radius="0.04" length="0.05"/>
+      </geometry>
+      <surface>
+        <friction>
+          <ode>
+            <mu>80</mu>
+            <mu2>80</mu2>
           </ode>
         </friction>
       </surface>
     </collision>
-    <visual name='caster_visual'>
-      <origin xyz="-0.15 0 -0.05" rpy=" 0 0 0"/>
-      <geometry>
-        <sphere radius="0.05"/>
-      </geometry>
-    </visual>
-  </link>
-  <link name="left_wheel">
-    <!--origin xyz="0.1 0.13 0.1" rpy="0 1.5707 1.5707"/-->
-    <collision name="collision">
-      <origin xyz="0 0 0" rpy="0 1.5707 1.5707"/>
-      <geometry>
-        <cylinder radius="0.1" length="0.05"/>
-      </geometry>
-    </collision>
     <visual name="left_wheel_visual">
       <origin xyz="0 0 0" rpy="0 1.5707 1.5707"/>
       <geometry>
-        <cylinder radius="0.1" length="0.05"/>
-      </geometry>
-    </visual>
-    <inertial>
-      <origin xyz="0 0 0" rpy="0 1.5707 1.5707"/>
-      <mass value="5"/>
-      <cylinder_inertia m="5" r="0.1" h="0.05"/>
+        <cylinder radius="0.04" length="0.04"/>
+      </geometry>
+    </visual>
+    <inertial>
+      <origin xyz="0 0 0" rpy="0 1.5707 1.5707"/>
+      <mass value="2"/>
+      <inertia
+        ixx="1.0" ixy="0.0" ixz="0.0"
+        iyy="1.0" iyz="0.0"
+        izz="1.0"/>
+    </inertial>
+  </link>
+  <link name="right_wheel_front">
+    <!--origin xyz="0.1 0.13 0.1" rpy="0 1.5707 1.5707"/-->
+    <collision name="collision">
+      <origin xyz="0 0 0" rpy="0 1.5707 1.5707"/>
+      <geometry>
+        <cylinder radius="0.04" length="0.05"/>
+      </geometry>
+      <surface>
+        <friction>
+          <ode>
+            <mu>10</mu>
+            <mu2>10</mu2>
+          </ode>
+        </friction>
+      </surface>
+    </collision>
+    <visual name="right_wheel_front_visual">
+      <origin xyz="0 0 0" rpy="0 1.5707 1.5707"/>
+      <geometry>
+        <cylinder radius="0.04" length="0.04"/>
+      </geometry>
+    </visual>
+    <inertial>
+      <mass value="4"/>
+      <origin xyz="0.0 0 0.0" rpy="0 0 0"/>
+      <inertia
+          ixx="1.0" ixy="0" ixz="0"
+          iyy="1.0" iyz="0"
+          izz="1.0"
+      />
+    </inertial>
+  </link>
+  <link name="right_wheel_middle">
+    <!--origin xyz="0.1 0.13 0.1" rpy="0 1.5707 1.5707"/-->
+    <collision name="collision">
+      <origin xyz="0 0 0.008" rpy="0 1.5707 1.5707"/>
+      <geometry>
+        <box size=".075 .18 .04"/>
+      </geometry>
+    </collision>
+    <visual name="right_wheel_middle_visual">
+      <origin xyz="0 0 0.008" rpy="0 1.5707 1.5707"/>
+      <geometry>
+        <box size=".075 .18 .04"/>
+      </geometry>
+    </visual>
+    <inertial>
+      <origin xyz="0 0 0" rpy="0 1.5707 1.5707"/>
+      <mass value="2"/>
       <inertia
         ixx="1.0" ixy="0.0" ixz="0.0"
@@ -74,21 +171,28 @@
   </link>
   <link name="right_wheel">
-    <!--origin xyz="0.1 -0.13 0.1" rpy="0 1.5707 1.5707"/-->
-    <collision name="collision">
-      <origin xyz="0 0 0" rpy="0 1.5707 1.5707"/>
-      <geometry>
-        <cylinder radius="0.1" length="0.05"/>
-      </geometry>
+    <!--origin xyz="0.1 0.13 0.1" rpy="0 1.5707 1.5707"/-->
+    <collision name="collision">
+      <origin xyz="0 0 0" rpy="0 1.5707 1.5707"/>
+      <geometry>
+        <cylinder radius="0.04" length="0.05"/>
+      </geometry>
+      <surface>
+        <friction>
+          <ode>
+            <mu>80</mu>
+            <mu2>80</mu2>
+          </ode>
+        </friction>
+      </surface>
     </collision>
     <visual name="right_wheel_visual">
       <origin xyz="0 0 0" rpy="0 1.5707 1.5707"/>
       <geometry>
-        <cylinder radius="0.1" length="0.05"/>
-      </geometry>
-    </visual>
-    <inertial>
-      <origin xyz="0 0 0" rpy="0 1.5707 1.5707"/>
-      <mass value="5"/>
-      <cylinder_inertia m="5" r="0.1" h="0.05"/>
+        <cylinder radius="0.04" length="0.04"/>
+      </geometry>
+    </visual>
+    <inertial>
+      <origin xyz="0 0 0" rpy="0 1.5707 1.5707"/>
+      <mass value="2"/>
       <inertia
         ixx="1.0" ixy="0.0" ixz="0.0"
@@ -113,3 +217,62 @@
     <joint_properties damping="0.0" friction="0.0"/>
   </joint>
+  <joint type="continuous" name="left_wheel_front_hinge">
+    <origin xyz="-0.1 0.15 0" rpy="0 0 0"/>
+    <child link="left_wheel_front"/>
+    <parent link="chassis"/>
+    <axis xyz="0 1 0" rpy="0 0 0"/>
+    <limit effort="100" velocity="100"/>
+    <joint_properties damping="0.0" friction="0.0"/>
+  </joint>
+  <joint type="fixed" name="left_wheel_middle_hinge">
+    <origin xyz="0 0.15 0.00" rpy="0 0 0"/>
+    <child link="left_wheel_middle"/>
+    <parent link="chassis"/>
+    <axis xyz="0 1 0" rpy="0 0 0"/>
+    <limit effort="100" velocity="100"/>
+    <joint_properties damping="0.0" friction="0.0"/>
+  </joint>
+  <joint type="continuous" name="right_wheel_front_hinge">
+    <origin xyz="-0.1 -0.15 0" rpy="0 0 0"/>
+    <child link="right_wheel_front"/>
+    <parent link="chassis"/>
+    <axis xyz="0 1 0" rpy="0 0 0"/>
+    <limit effort="100" velocity="100"/>
+    <joint_properties damping="0.0" friction="0.0"/>
+  </joint>
+  <joint type="fixed" name="right_wheel_middle_hinge">
+    <origin xyz="0 -0.15 0.00" rpy="0 0 0"/>
+    <child link="right_wheel_middle"/>
+    <parent link="chassis"/>
+    <axis xyz="0 1 0" rpy="0 0 0"/>
+    <limit effort="100" velocity="100"/>
+    <joint_properties damping="0.0" friction="0.0"/>
+  </joint>
+  <link name="camera">
+    <collision>
+      <origin xyz="0 0 0" rpy="0 0 0"/>
+      <geometry>
+        <box size="${cameraSize} ${cameraSize} ${cameraSize}"/>
+      </geometry>
+    </collision>
+    <visual>
+      <origin xyz="0 0 0" rpy="0 0 0"/>
+      <geometry>
+        <box size="${cameraSize} ${cameraSize} ${cameraSize}"/>
+      </geometry>
+      <material name="green"/>
+    </visual>
+    <inertial>
+      <mass value="${cameraMass}" />
+      <origin xyz="0 0 0" rpy="0 0 0"/>
+      <box_inertia m="${cameraMass}" x="${cameraSize}" y="${cameraSize}" z="${cameraSize}" />
+      <inertia ixx="1e-6" ixy="0" ixz="0" iyy="1e-6" iyz="0" izz="1e-6" />
+    </inertial>
+  </link>
+  <joint name="camera_joint" type="fixed">
+    <axis xyz="0.18 1 0" />
+    <origin xyz="-0.08 0 0.1" rpy="0 0 0"/>
+    <parent link="chassis"/>
+    <child link="camera"/>
+  </joint>
 </robot>

Commit message: update opencv_vision

File: src/robot_description/urdf/robot.xacro (robot description, xacro)
@@ -251,5 +251,5 @@
   <link name="camera">
     <collision>
-      <origin xyz="0 0 0" rpy="0 0 0"/>
+      <origin xyz="0 0 0" rpy="0 0 -3.1415"/>
       <geometry>
         <box size="${cameraSize} ${cameraSize} ${cameraSize}"/>
@@ -257,5 +257,5 @@
     </collision>
     <visual>
-      <origin xyz="0 0 0" rpy="0 0 0"/>
+      <origin xyz="0 0 0" rpy="0 0 -3.1415"/>
       <geometry>
         <box size="${cameraSize} ${cameraSize} ${cameraSize}"/>
@@ -265,5 +265,5 @@
     <inertial>
       <mass value="${cameraMass}" />
-      <origin xyz="0 0 0" rpy="0 0 0"/>
+      <origin xyz="0 0 0" rpy="0 0 -3.1415"/>
       <box_inertia m="${cameraMass}" x="${cameraSize}" y="${cameraSize}" z="${cameraSize}" />
       <inertia ixx="1e-6" ixy="0" ixz="0" iyy="1e-6" iyz="0" izz="1e-6" />
@@ -272,5 +272,5 @@
   <joint name="camera_joint" type="fixed">
     <axis xyz="0.18 1 0" />
-    <origin xyz="-0.08 0 0.1" rpy="0 0 0"/>
+    <origin xyz="-0.11 0 0.1" rpy="0 0 -3.1415"/>
     <parent link="chassis"/>
     <child link="camera"/>
